Commit message: Fixed paths so they are always easy to find

File: models/habitat_demonstration_unit/urdf/habitat_demonstration_unit.urdf.xacro (robot description, xacro)
@@ -24,5 +24,5 @@
       <origin xyz="0 0 0" rpy="0 0 0" />
       <geometry>
-        <mesh filename="package://space_resources/models/habitat_demonstration_unit/meshes/habitat_demonstration_unit_part_1.dae" scale="1 1 1"/>
+        <mesh filename="file://$(find space_resources)/models/habitat_demonstration_unit/meshes/habitat_demonstration_unit_part_1.dae" scale="1 1 1"/>
       </geometry>
     </visual>
@@ -30,5 +30,5 @@
       <origin xyz="0 0 0" rpy="0 0 0"/>
       <geometry>
-        <mesh filename="package://space_resources/models/habitat_demonstration_unit/meshes/habitat_demonstration_unit_part_1.dae" scale="1 1 1"/>
+        <mesh filename="file://$(find space_resources)/models/habitat_demonstration_unit/meshes/habitat_demonstration_unit_part_1.dae" scale="1 1 1"/>
       </geometry>
     </collision>

File: models/htv_transfer_vehicle/urdf/htv1_external_pallet.macro.xacro (robot description, xacro)
@@ -12,5 +12,5 @@
        <origin xyz="0 0 0" rpy="0 0 0" />
        <geometry>
-         <mesh filename="package://space_resources/models/htv_transfer_vehicle/meshes/htv_ep1a_1_100_v01_textured.dae" scale="1 1 1"/>
+         <mesh filename="file://$(find space_resources)/models/htv_transfer_vehicle/meshes/htv_ep1a_1_100_v01_textured.dae" scale="1 1 1"/>
        </geometry>
      </visual>
@@ -18,5 +18,5 @@
        <origin xyz="0 0 0" rpy="0 0 0"/>
        <geometry>
-         <mesh filename="package://space_resources/models/htv_transfer_vehicle/meshes/htv_ep1a_1_100_v01_textured.dae" scale="1 1 1"/>
+         <mesh filename="file://$(find space_resources)/models/htv_transfer_vehicle/meshes/htv_ep1a_1_100_v01_textured.dae" scale="1 1 1"/>
        </geometry>
      </collision>

File: models/htv_transfer_vehicle/urdf/htv1_module.macro.xacro (robot description, xacro)
@@ -12,5 +12,5 @@
        <origin xyz="0 0 0" rpy="0 0 0" />
        <geometry>
-         <mesh filename="package://space_resources/models/htv_transfer_vehicle/meshes/htv_1_100_v01_textured.dae" scale="1 1 1"/>
+         <mesh filename="file://$(find space_resources)/models/htv_transfer_vehicle/meshes/htv_1_100_v01_textured.dae" scale="1 1 1"/>
        </geometry>
      </visual>
@@ -18,5 +18,5 @@
        <origin xyz="0 0 0" rpy="0 0 0"/>
        <geometry>
-         <mesh filename="package://space_resources/models/htv_transfer_vehicle/meshes/htv_1_100_v01_textured.dae" scale="1 1 1"/>
+         <mesh filename="file://$(find space_resources)/models/htv_transfer_vehicle/meshes/htv_1_100_v01_textured.dae" scale="1 1 1"/>
        </geometry>
      </collision>
