Commit message: Set builder mesh

File: models/habitat_demonstration_unit/urdf/habitat_demonstration_unit_open_top.urdf.xacro (robot description, xacro)
@@ -24,5 +24,6 @@
       <origin xyz="0 0 0" rpy="0 0 0" />
       <geometry>
-        <mesh filename="file://$(find space_resources)/models/habitat_demonstration_unit/meshes/habitat_demonstration_unit_part_1_open_top.dae" scale="1 1 1"/>
+        <!--<mesh filename="file://$(find space_resources)/models/habitat_demonstration_unit/meshes/habitat_demonstration_unit_part_1_open_top.dae" scale="1 1 1"/>-->
+            <mesh filename="file://$(find space_resources)/models/habitat_demonstration_unit/meshes/hdu_builder.dae" scale="1 1 1"/>
       </geometry>
     </visual>
@@ -30,5 +31,6 @@
       <origin xyz="0 0 0" rpy="0 0 0"/>
       <geometry>
-        <mesh filename="file://$(find space_resources)/models/habitat_demonstration_unit/meshes/habitat_demonstration_unit_part_1_open_top.dae" scale="1 1 1"/>
+        <!--<mesh filename="file://$(find space_resources)/models/habitat_demonstration_unit/meshes/habitat_demonstration_unit_part_1_open_top.dae" scale="1 1 1"/>-->
+            <mesh filename="file://$(find space_resources)/models/habitat_demonstration_unit/meshes/hdu_builder.dae" scale="1 1 1"/>
       </geometry>
     </collision>

Commit message: working demo fro builder-11 spot inspection

File: models/habitat_demonstration_unit/urdf/habitat_demonstration_unit_open_top.urdf.xacro (robot description, xacro)
@@ -24,5 +24,5 @@
       <origin xyz="0 0 0" rpy="0 0 0" />
       <geometry>
-        <mesh filename="file://$(find space_resources)/models/habitat_demonstration_unit/meshes/habitat_demonstration_unit_part_1_open_top.dae" scale="1 1 1"/>
+        <mesh filename="file://$(find space_resources)/models/habitat_demonstration_unit/meshes/habitat_demonstration_unit_part_1_open_top_solidified.dae" scale="1 1 1"/>
       </geometry>
     </visual>
@@ -30,5 +30,5 @@
       <origin xyz="0 0 0" rpy="0 0 0"/>
       <geometry>
-        <mesh filename="file://$(find space_resources)/models/habitat_demonstration_unit/meshes/habitat_demonstration_unit_part_1_open_top.dae" scale="1 1 1"/>
+        <mesh filename="file://$(find space_resources)/models/habitat_demonstration_unit/meshes/habitat_demonstration_unit_part_1_open_top_solidified.dae" scale="1 1 1"/>
       </geometry>
     </collision>
